File: HARDWARE/The Flying Jalapeno v01.sch (EAGLE design)
At the start: 80 parts, among them J1 ., J2 7V, Q1 16MHZ, Q2 MMBT2222A, Q3 P-Channel MOSFET, Q4 MMBT2222A, Q5 P-Channel MOSFET, U2 ATMEGA328P_TQFP

Commit message: more prod ids
Parts:
- Q3, Q5: device Testing:MOSFET-PCHANNELPTH -> SparkFun-DiscreteSemi:MOSFET-PCHANNELNDP6020P_20V_24A_LOW_VGS_TH
Other:
- note removed: "TRANS-13060"
Changed lines of the file:
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@@
 <part name="R11" library="SparkFun-Resistors" deviceset="100OHM-1/10W-1%(0603)" device="" value="100"/>
 <part name="GND15" library="SparkFun" deviceset="GND" device=""/>
-<part name="Q3" library="Testing" deviceset="MOSFET-PCHANNEL" device="PTH" value="P-Channel MOSFET"/>
+<part name="Q3" library="SparkFun-DiscreteSemi" deviceset="MOSFET-PCHANNEL" device="NDP6020P_20V_24A_LOW_VGS_TH" value="P-Channel MOSFET"/>
 <part name="C3" library="SparkFun-Capacitors" deviceset="100UF-63V-20%(ELECT)" device="" value="100uF"/>
 <part name="GND16" library="SparkFun" deviceset="GND" device=""/>
@@
 <part name="R14" library="SparkFun-Resistors" deviceset="100OHM-1/10W-1%(0603)" device="" value="100"/>
 <part name="GND17" library="SparkFun" deviceset="GND" device=""/>
-<part name="Q5" library="Testing" deviceset="MOSFET-PCHANNEL" device="PTH" value="P-Channel MOSFET"/>
+<part name="Q5" library="SparkFun-DiscreteSemi" deviceset="MOSFET-PCHANNEL" device="NDP6020P_20V_24A_LOW_VGS_TH" value="P-Channel MOSFET"/>
 <part name="C8" library="SparkFun-Capacitors" deviceset="100UF-63V-20%(ELECT)" device="" value="100uF"/>
 <part name="GND18" library="SparkFun" deviceset="GND" device=""/>
@@
 <plain>
 <text x="347.98" y="266.7" size="3.81" layer="94">PRETESTS</text>
-<text x="150.622" y="199.39" size="1.778" layer="97" rot="MR0">TRANS-13060</text>
 <text x="139.954" y="196.088" size="0.8128" layer="94">S</text>
 <text x="145.288" y="188.722" size="0.8128" layer="94">G</text>
 <text x="149.098" y="196.088" size="0.8128" layer="94">D</text>
-<text x="158.242" y="135.89" size="1.778" layer="97" rot="MR0">TRANS-13060</text>
 <text x="145.034" y="132.588" size="0.8128" layer="94">S</text>
 <text x="150.368" y="125.222" size="0.8128" layer="94">G</text>
@@
 <instance part="GND15" gate="1" x="144.78" y="162.56"/>
 <instance part="Q3" gate="G$1" x="144.78" y="195.58" smashed="yes" rot="MR90">
-<attribute name="NAME" x="145.542" y="204.47" size="1.778" layer="95" rot="MR0"/>
-<attribute name="VALUE" x="155.702" y="201.93" size="1.778" layer="96" rot="MR0"/>
+<attribute name="NAME" x="146.558" y="200.152" size="1.778" layer="95" rot="MR0"/>
 </instance>
 <instance part="C3" gate="G$1" x="124.46" y="190.5"/>
@@
 <instance part="R14" gate="G$1" x="137.16" y="109.22"/>
 <instance part="GND17" gate="1" x="149.86" y="99.06"/>
-<instance part="Q5" gate="G$1" x="149.86" y="132.08" smashed="yes" rot="MR90">
-<attribute name="NAME" x="153.162" y="140.97" size="1.778" layer="95" rot="MR0"/>
-<attribute name="VALUE" x="163.322" y="138.43" size="1.778" layer="96" rot="MR0"/>
-</instance>
+<instance part="Q5" gate="G$1" x="149.86" y="132.08" smashed="yes" rot="MR90"/>
 <instance part="C8" gate="G$1" x="129.54" y="127"/>
 <instance part="GND18" gate="1" x="129.54" y="116.84"/>

Commit message: more prod ids and some sch cleanup
last thing that needs prod ids is the headers at the bottom, not sure if
we're gonna go with break away or combining 10pin and 8pin pieces
Parts:
- Q2, Q4: value MMBT2222A -> (none)
- Q5: value P-Channel MOSFET -> MOSFET-PCHANNELNDP6020P_20V_24A_LOW_VGS_TH
- R26, R27: value 22M ohm -> 22M; device SparkFun-Resistors:330OHM1/10W1%(0603) -> SparkFun-Resistors:22MOHM-1/10W-10%(0603)
Other:
- note removed: "RES-11132"
- moved on the sheet: C1, C17, C18, C2, D1, D3, D4, J1, Q1, R2, R20, R5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
