File: HARDWARE/The Flying Jalapeno v01.sch (EAGLE design)
At the start: 80 parts, among them J1 ., J2 7V, Q1 16MHZ, Q3 P-Channel MOSFET, Q5 MOSFET-PCHANNELNDP6020P_20V_2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, U2 ATMEGA328P_TQFP

Commit message: Moved to Mega2560 and 2x30 2mm connector
device and packages for the 2x30 connector all live in the "local"
sparkfun.lbr for now. I will push to testing.lbr soon.
Parts:
- removed C12, C16, C7: 0.1uF, SparkFun-Capacitors:0.1UF-25V(+80/-20%)(0603)
- removed D2: RED, SparkFun-LED:LED-RED1206
- removed J1: ., SparkFun:AVR_SPI_PRG_62X3_LOCK
- removed JP1: FTDI Basic, SparkFun-Connectors:ARDUINO_SERIAL_PROGRAMSMD
- removed JP4: FLYING_JALAPENO, Testing:FLYING_JALAPENO
- removed SJ3, SJ4: JUMPER-PAD-3-2OF3_NC_BY_PASTE, SparkFun-Passives:JUMPER-PAD-3-2OF3_NC_BY_PASTE
- removed U2: ATMEGA328P_TQFP, SparkFun-DigitalIC:ATMEGA328P_TQFP
- added C19, C21, C22: 0.1uF, SparkFun-Capacitors:0.1UF-25V(+80/-20%)(0603)
- added D6: RED, SparkFun-LED:LED-RED1206
- added JP15: FTDI, SparkFun:ARDUINO_SERIAL_PROGRAMSMD
- added JP3: AVR_SPI_PRG_6PTH, SparkFun:AVR_SPI_PRG_6PTH
- added JP6: FLYING_JALAPENO_V2FEMALE, SparkFun:FLYING_JALAPENO_V2FEMALE
- added Q6, Q7: 200mA/50V, SparkFun-DiscreteSemi:MOSFET-NCHANNELBSS138
- added R31, R32: DNP, SparkFun-Resistors:10KOHM-1/10W-1%(0603)0603
- added R33: 390, SparkFun-Resistors:390OHM1/10W1%(0603)
- added R34, R35, R36, R41: 10K, SparkFun-Resistors:10KOHM-1/10W-1%(0603)0603
- added R37, R38: ?, SparkFun-Resistors:390OHM1/10W1%(0603)
- added R39: 100k, SparkFun-Resistors:100KOHM-1/10W-1%(0603)
- added STANDOFF1, STANDOFF2, STANDOFF3, STANDOFF4: STAND-OFFTIGHT, SparkFun-Electromechanical:STAND-OFFTIGHT
- added U4: ATMEGA2560AU, SparkFun:ATMEGA2560AU
- R17: value 390 -> 10K; device SparkFun-Resistors:390OHM1/10W1%(0603) -> SparkFun-Resistors:10KOHM-1/10W-1%(0603)0603
Connections:
- removed net A6/PRETESTREAD_V1: JP4.PC6(ADC6), R13.2, R3.1, R9.2, U2.ADC6
- removed net A7/PRETESTREAD_V2: JP4.PC7(ADC7), R28.1, R29.2, R30.2, U2.ADC7
- removed net CAPSENSE1: JP4.CAPSENSE1(D7), R26.2
- removed net CAPSENSE2: JP4.CAPSENSE2(D8), R27.2
- removed net D10/CONT1: JP4.PB2(SS/OC1B), R11.1, R22.1, U2.PB2(SS/OC1B)
- removed net D11/CONT2: J1.4, JP4.PB3(MOSI/OC2), R14.1, U2.PB3(MOSI/OC2)
- removed net D12/PRETEST-WRITE: J1.1, JP4.PB4(MISO), R13.1, R30.1, U2.PB4(MISO)
- removed net FAIL: JP4.FAIL(D6), R25.2
- removed net N$4 (its old number): IC2.ADJ, R4.1, SJ3.2
- removed net PASS: JP4.PASS(D5), R24.2
- removed net PT-FAIL: JP4.PT-FAIL(D4), R23.2
- removed net PT-PASS: JP4.PT-PASS(D10), R22.2
- removed net RX: JP1.RXI, JP4.PD1(TXD), U2.PD1(TXD)
- removed net SCK: J1.3, JP4.PB5(SCK), R6.1, U2.PB5(SCK)
- removed net TX: JP1.TXO, JP4.PD0(RXD), U2.PD0(RXD)
- new net 31/CAPRETURN2: R27.1, U4.(A14)PC6
- new net 33/V1_3.3V: R7.1, U4.(A12)PC4
- new net 34/RAW_PASS_LED: R33.1, U4.(A11)PC3
- new net 35/V1_5V: R1.1, U4.(A10)PC2
- new net 36/V2_3.3V: R8.1, U4.(A9)PC1
- new net 37/V2_3.7V: R38.1, U4.(A8)PC0
- new net 38/V2_4.2V: R37.1, U4.(T0)PD7
- new net 39/V2_5V: R21.1, U4.(ALE)PG2
- new net 40/FAIL: R25.2, U4.(RD)PG1
- new net 41/PASS: R24.2, U4.(WR)PG0
- new net 42/PT_FAIL: R23.2, U4.PL7
- new net 43/PT_PASS: R22.2, U4.PL6
- new net 44/PT_CTRL: R13.1, R30.1, U4.PL5(OC5C)
- new net 45/CAPSENSE1: JP6.45/CAPSENSE1, U4.PL4(OC5B)
- new net 46/CAPSENSE2: JP6.46/CAPSENSE2, U4.PL3(OC5A)
- new net 47/CAPRETURN1: R26.1, U4.PL2(T5)
- new net 48/PWR_CTRL1: R11.1, U4.PL1(ICP5)
- new net 49/PWR_CTRL2: R14.1, U4.PL0(ICP4)
- new net A10: JP6.A10, U4.PK2(ADC10/PCINT18)
- new net A11: JP6.A11, U4.PK3(ADC11/PCINT19)
- new net A12: JP6.A12, U4.PK4(ADC12/PCINT20)
- new net A13/RAW_READ: R36.2, R39.1, U4.PK5(ADC13/PCINT21)
- new net A14/PT_READ_V1: R13.2, R3.1, R9.2, U4.PK6(ADC14/PCINT22)
- new net A15/PT_READ_V2: R28.1, R29.2, R30.2, U4.PK7(ADC15/PCINT23)
- new net A6: JP6.A6, U4.(ADC6/TDO)PF6
- new net A7: JP6.A7, U4.(ADC7/TDI)PF7
- new net A8: JP6.A8, U4.PK0(ADC8/PCINT16)
- new net A9: JP6.A9, U4.PK1(ADC9/PCINT17)
- new net D10: JP6.10, U4.(OC2A/PCINT4)PB4
- new net D11: JP6.11, U4.(OC1A/PCINT5)PB5
- new net D12: JP6.12, U4.(OC1B/PCINT6)PB6
- new net D13: JP6.13, R6.1, U4.(OC0A/OC1C/PCINT7)PB7
- new net D22: JP6.22, U4.(AD0)PA0
- new net D23: JP6.23, U4.(AD1)PA1
- new net D24: JP6.24, U4.(AD2)PA2
- new net D25: JP6.25, U4.(AD3)PA3
- new net D26: JP6.26, U4.(AD4)PA4
- new net D27: JP6.27, U4.(AD5)PA5
- new net D28: JP6.28, U4.(AD6)PA6
- new net D29: JP6.29, U4.(AD7)PA7
- new net D30: JP6.30, U4.(A15)PC7
- new net FTDI_VCC: JP15.VCC, Q6.G, Q7.G, R34.2, R41.2
- new net N$25: D6.A, R33.2
- new net N$26: JP15.RXI, Q6.S, R41.1
- new net N$7: JP6.42/PT_FAIL, R23.1
- new net N$73: Q1.3, U4.XTAL2
- new net N$74: Q1.1, U4.XTAL1
- new net PB0: JP6.53, U4.(SS/PCINT0)PB0
- new net PB1: JP3.3, JP6.52, U4.(SCK/PCINT1)PB1
- new net PB2: JP3.4, JP6.51, U4.(MOSI/PCINT2)PB2
- new net PB3: JP3.1, JP6.50, U4.(MISO/PCINT3)PB3
- new net PC5: U4.(A13)PC5
- new net RX0: Q7.D, R35.1, U4.(RXD0/PCIN8)PE0
- new net RX1: JP6.19(RX1/INT4), U4.(RXD1/INT2)PD2
- new net RX2: JP6.17(RX2), U4.PH0(RXD2)
- new net RX3: JP6.15(RX3), U4.PJ0(RXD3/PCINT9)
- new net SCL: JP6.21(SCL/INT2), R32.1, U4.(SCL/INT0)PD0
- new net SDA: JP6.20(SDA/INT3), R31.1, U4.(SDA/INT1)PD1
- new net TX0: Q6.D, R17.1, U4.(TXD0)PE1
- new net TX1: JP6.18(TX1/INT5), U4.(TXD1/INT3)PD3
- new net TX2: JP6.16(TX2), U4.PH1(TXD2)
- new net TX3: JP6.14(TX3), U4.PJ1(TXD3/PCINT10)
- net A0: now also JP6.A0(RX0), U4.(ADC0)PF0; no longer JP4.PC0(ADC0), U2.PC0(ADC0)
- net A1: now also JP6.A1(TX0), U4.(ADC1)PF1; no longer JP4.PC1(ADC1), U2.PC1(ADC1)
- net A2: now also JP6.A2, U4.(ADC2)PF2; no longer JP4.PC2(ADC2), U2.PC2(ADC2)
- net A3: now also JP6.A3, U4.(ADC3)PF3; no longer JP4.PC3(ADC3), U2.PC3(ADC3)
- net A4: now also JP6.A4, U4.(ADC4/TCK)PF4; no longer JP4.PC4(ADC4/SDA), U2.PC4(ADC4/SDA)
- net A5: now also JP6.A5, U4.(ADC5/TMS)PF5; no longer JP4.PC5(ADC5/SCL), U2.PC5(ADC5/SCL)
- net AREF: now also U4.AREF; no longer U2.AREF
- net D2: now also JP6.2(INT0), U4.(OC3B/INT4)PE4; no longer JP4.PD2(INT0), U2.PD2(INT0)
- net D3: now also JP6.3(INT1), U4.(OC3C/INT5)PE5; no longer JP4.PD3(INT1), U2.PD3(INT1)
- net D4: now also JP6.4, U4.(OC0B)PG5; no longer JP4.PD4(XCK/T0), R23.1, U2.PD4(XCK/T0)
- net D5: now also JP6.5, U4.(OC3A/AIN1)PE3; no longer JP4.PD5(T1), R24.1, U2.PD5(T1)
- net D6: now also JP6.6, U4.PH3(OC4A); no longer JP4.PD6(AIN0), R25.1, U2.PD6(AIN0)
- net D7: now also JP6.7, U4.PH4(OC4B); no longer JP4.PD7(AIN1), R26.1, U2.PD7(AIN1)
- net D8: now also JP6.8, U4.PH5(OC4C); no longer JP4.PB0(ICP), R27.1, U2.PB0(ICP)
- net D9: now also JP6.9, U4.PH6(OC2B); no longer JP4.PB1(OC1A), U2.PB1(OC1A)
- net DTR: now also JP15.DTR; no longer JP1.DTR
- net GND: now also C19.1, C21.1, C22.1, D6.C, JP15.CTS, JP15.GND, JP3.6, JP6.GND, R36.1, U4.AGND, U4.GND, U4.GND1, U4.GND2, U4.GND3; no longer C12.2, C16.2, C7.2, D2.C, J1.6, JP1.CTS, JP1.GND, JP4.GND, R1.1, R21.1, R7.1, R8.1, U2.AGND, U2.GND@3, U2.GND@5
- net N$1: now also JP6.47/CAPRETURN1, R26.2; no longer Q1.1, U2.PB7(XTAL2/TOSC2)
- net N$10: now also R21.2, R37.2, R38.2, R8.2; no longer SJ4.2
- net N$16: now also JP15.TXO, Q7.S, R34.1; no longer D2.A, R17.1
- net N$19: now also JP6.41/PASS, R24.1; no longer R21.2, SJ4.1
- net N$2: now also JP6.31/CAPRETURN2, R27.2; no longer Q1.3, U2.PB6(XTAL1/TOSC1)
- net N$20: now also JP6.40/FAIL, R25.1; no longer R8.2, SJ4.3
- net N$21: no longer C7.1
- net N$6: now also JP6.43/PT_PASS, R22.1; no longer R7.2, SJ3.1
- net N$9: now also IC2.ADJ, R4.1, R7.2; no longer SJ3.3
- net RAW: now also R39.2; no longer JP4.RAW
- net RESET: now also JP3.5, U4.RESET; no longer J1.5, U2.PC6(/RESET)
- net V1: now also JP6.V1; no longer JP4.V1
- net V2: now also JP6.V2; no longer JP4.V2
- net VCC: now also C19.2, C21.2, C22.2, JP3.2, R31.2, R32.2, R35.2, U4.AVCC, U4.VCC, U4.VCC1, U4.VCC2, U4.VCC3; no longer C12.1, J1.2, JP4.VCC, U2.AVCC, U2.VCC@4, U2.VCC@6
- net VREG2OUT: no longer C16.1
Other:
- note added: "ATMEGA2560V"
- note added: "RAW SPLIT"
- note added: "V1 (3.3 or 5)"
- note added: "V2 (3.3, 3.7, 4.2, 5)"
- note removed: "CAPSENSE RESISTORS"
- note removed: "CONNECTION TO POGOBED (2x18 header)"
- note removed: "LED RESISTORS"
- note removed: "V1 (default:5V)"
- note removed: "V2 (default:3.3V)"

Commit message: Modified Capsense pad device to use only 1 pin/pad
I realized that I don't need the usual two lines for capsense buttons on
this (SEND/RETURN). Because the resistors are going to live on the
board, then the "button" on the testbed is only an extension of one net.
Updated library devices to reflect this correction.
Parts:
- R38: value ? -> 470; device SparkFun-Resistors:390OHM1/10W1%(0603) -> SparkFun-Resistors:470OHM1/10W1%(0603)
Connections:
- removed net N$1: JP6.47/CAPRETURN1, R26.2
- removed net N$2: JP6.31/CAPRETURN2, R27.2
- net 45/CAPSENSE1: now also JP6.CAP_PAD1, R26.2; no longer JP6.45/CAPSENSE1
- net 46/CAPSENSE2: now also JP6.CAP_PAD2, R27.2; no longer JP6.46/CAPSENSE2
- net RAW: now also JP6.RAW
Other:
- moved on the sheet: R26, R27
Changed lines of the file:
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@@
 <layer number="112" name="tSilk" color="7" fill="1" visible="yes" active="yes"/>
 <layer number="113" name="IDFDebug" color="4" fill="1" visible="yes" active="yes"/>
+<layer number="114" name="Badge_Outline" color="11" fill="1" visible="no" active="no"/>
 <layer number="116" name="Patch_BOT" color="9" fill="4" visible="yes" active="yes"/>
 <layer number="118" name="Rect_Pads" color="7" fill="1" visible="yes" active="yes"/>
@@
 <part name="GND38" library="SparkFun" deviceset="GND" device=""/>
 <part name="R37" library="SparkFun-Resistors" deviceset="390OHM1/10W1%(0603)" device="" value="?"/>
-<part name="R38" library="SparkFun-Resistors" deviceset="390OHM1/10W1%(0603)" device="" value="?"/>
+<part name="R38" library="SparkFun-Resistors" deviceset="470OHM1/10W1%(0603)" device="" value="470"/>
 <part name="R39" library="SparkFun-Resistors" deviceset="100KOHM-1/10W-1%(0603)" device="" value="100k"/>
 <part name="C19" library="SparkFun-Capacitors" deviceset="0.1UF-25V(+80/-20%)(0603)" device="" value="0.1uF"/>
@@
 <instance part="P+7" gate="G$1" x="91.44" y="20.32"/>
 <instance part="JP6" gate="G$1" x="505.46" y="180.34"/>
-<instance part="GND54" gate="1" x="477.52" y="124.46"/>
-<instance part="R26" gate="G$1" x="538.48" y="144.78" smashed="yes" rot="R180">
-<attribute name="NAME" x="535.59" y="145.7814" size="0.8128" layer="95" rot="R180"/>
-<attribute name="VALUE" x="543.49" y="144.482" size="0.8128" layer="96" rot="R180"/>
-</instance>
-<instance part="R27" gate="G$1" x="538.48" y="185.42" smashed="yes" rot="R180">
-<attribute name="NAME" x="535.99" y="186.5214" size="0.8128" layer="95" rot="R180"/>
-<attribute name="VALUE" x="543.49" y="185.122" size="0.8128" layer="96" rot="R180"/>
+<instance part="GND54" gate="1" x="477.52" y="121.92"/>
+<instance part="R26" gate="G$1" x="541.02" y="147.32" smashed="yes" rot="R180">
+<attribute name="NAME" x="538.13" y="148.3214" size="0.8128" layer="95" rot="R180"/>
+<attribute name="VALUE" x="546.03" y="147.022" size="0.8128" layer="96" rot="R180"/>
+</instance>
+<instance part="R27" gate="G$1" x="541.02" y="142.24" smashed="yes" rot="R180">
+<attribute name="NAME" x="538.53" y="143.3414" size="0.8128" layer="95" rot="R180"/>
+<attribute name="VALUE" x="546.03" y="141.942" size="0.8128" layer="96" rot="R180"/>
 </instance>
 <instance part="R22" gate="G$1" x="538.48" y="154.94" smashed="yes">
@@
 <segment>
 <pinref part="GND54" gate="1" pin="GND"/>
-<wire x1="477.52" y1="129.54" x2="477.52" y2="127" width="0.1524" layer="91"/>
-<wire x1="480.06" y1="129.54" x2="477.52" y2="129.54" width="0.1524" layer="91"/>
+<wire x1="477.52" y1="127" x2="477.52" y2="124.46" width="0.1524" layer="91"/>
+<wire x1="480.06" y1="127" x2="477.52" y2="127" width="0.1524" layer="91"/>
 <pinref part="JP6" gate="G$1" pin="GND"/>
 </segment>
@@
 <pinref part="R39" gate="G$1" pin="2"/>
 </segment>
+<segment>
+<pinref part="JP6" gate="G$1" pin="RAW"/>
+<wire x1="480.06" y1="231.14" x2="477.52" y2="231.14" width="0.1524" layer="91"/>
+<label x="477.52" y="231.14" size="1.27" layer="95" rot="R180" xref="yes"/>
+</segment>
 </net>
 <net name="A5" class="0">
@@
 </segment>
 <segment>
-<wire x1="530.86" y1="149.86" x2="533.4" y2="149.86" width="0.1524" layer="91"/>
-<pinref part="JP6" gate="G$1" pin="45/CAPSENSE1"/>
-<label x="533.4" y="149.86" size="1.27" layer="95" xref="yes"/>
+<label x="548.64" y="149.86" size="1.27" layer="95" xref="yes"/>
+<wire x1="533.4" y1="149.86" x2="548.64" y2="149.86" width="0.1524" layer="91"/>
+<pinref part="R26" gate="G$1" pin="2"/>
+<wire x1="533.4" y1="147.32" x2="535.94" y2="147.32" width="0.1524" layer="91"/>
+<wire x1="533.4" y1="149.86" x2="533.4" y2="147.32" width="0.1524" layer="91"/>
+<pinref part="JP6" gate="G$1" pin="CAP_PAD1"/>
+<wire x1="533.4" y1="147.32" x2="530.86" y2="147.32" width="0.1524" layer="91"/>
+<junction x="533.4" y="147.32"/>
 </segment>
 </net>
@@
 </segment>
 <segment>
-<wire x1="530.86" y1="147.32" x2="533.4" y2="147.32" width="0.1524" layer="91"/>
-<pinref part="JP6" gate="G$1" pin="46/CAPSENSE2"/>
-<label x="533.4" y="147.32" size="1.27" layer="95" xref="yes"/>
+<label x="548.64" y="144.78" size="1.27" layer="95" xref="yes"/>
+<pinref part="R27" gate="G$1" pin="2"/>
+<wire x1="533.4" y1="144.78" x2="548.64" y2="144.78" width="0.1524" layer="91"/>
+<wire x1="533.4" y1="142.24" x2="535.94" y2="142.24" width="0.1524" layer="91"/>
+<wire x1="533.4" y1="144.78" x2="533.4" y2="142.24" width="0.1524" layer="91"/>
+<pinref part="JP6" gate="G$1" pin="CAP_PAD2"/>
+<wire x1="533.4" y1="144.78" x2="530.86" y2="144.78" width="0.1524" layer="91"/>
+<junction x="533.4" y="144.78"/>
 </segment>
 </net>
@@
 <segment>
 <pinref part="R26" gate="G$1" pin="1"/>
-<wire x1="543.56" y1="144.78" x2="546.1" y2="144.78" width="0.1524" layer="91"/>
-<label x="546.1" y="144.78" size="1.27" layer="95" xref="yes"/>
+<wire x1="546.1" y1="147.32" x2="548.64" y2="147.32" width="0.1524" layer="91"/>
+<label x="548.64" y="147.32" size="1.27" layer="95" xref="yes"/>
 </segment>
 </net>
@@
 </segment>
 <segment>
-<label x="546.1" y="185.42" size="1.27" layer="95" xref="yes"/>
+<label x="548.64" y="142.24" size="1.27" layer="95" xref="yes"/>
 <pinref part="R27" gate="G$1" pin="1"/>
-<wire x1="543.56" y1="185.42" x2="546.1" y2="185.42" width="0.1524" layer="91"/>
+<wire x1="546.1" y1="142.24" x2="548.64" y2="142.24" width="0.1524" layer="91"/>
 </segment>
 </net>
@@
 </segment>
 <segment>
-<wire x1="530.86" y1="129.54" x2="533.4" y2="129.54" width="0.1524" layer="91"/>
+<wire x1="530.86" y1="127" x2="533.4" y2="127" width="0.1524" layer="91"/>
 <pinref part="JP6" gate="G$1" pin="53"/>
-<label x="533.4" y="129.54" size="1.27" layer="95" xref="yes"/>
+<label x="533.4" y="127" size="1.27" layer="95" xref="yes"/>
 </segment>
 </net>
@@
 </segment>
 <segment>
-<wire x1="530.86" y1="132.08" x2="533.4" y2="132.08" width="0.1524" layer="91"/>
+<wire x1="530.86" y1="129.54" x2="533.4" y2="129.54" width="0.1524" layer="91"/>
 <pinref part="JP6" gate="G$1" pin="52"/>
-<label x="533.4" y="132.08" size="1.27" layer="95" xref="yes"/>
+<label x="533.4" y="129.54" size="1.27" layer="95" xref="yes"/>
 </segment>
 </net>
@@
 </segment>
 <segment>
-<wire x1="530.86" y1="134.62" x2="533.4" y2="134.62" width="0.1524" layer="91"/>
+<wire x1="530.86" y1="132.08" x2="533.4" y2="132.08" width="0.1524" layer="91"/>
 <pinref part="JP6" gate="G$1" pin="51"/>
-<label x="533.4" y="134.62" size="1.27" layer="95" xref="yes"/>
+<label x="533.4" y="132.08" size="1.27" layer="95" xref="yes"/>
 </segment>
 </net>
@@
 </segment>
 <segment>
-<wire x1="530.86" y1="137.16" x2="533.4" y2="137.16" width="0.1524" layer="91"/>
+<wire x1="530.86" y1="134.62" x2="533.4" y2="134.62" width="0.1524" layer="91"/>
 <pinref part="JP6" gate="G$1" pin="50"/>
-<label x="533.4" y="137.16" size="1.27" layer="95" xref="yes"/>
+<label x="533.4" y="134.62" size="1.27" layer="95" xref="yes"/>
 </segment>
 </net>
@@
 <pinref part="D3" gate="G$1" pin="A"/>
 <wire x1="368.3" y1="228.6" x2="370.84" y2="228.6" width="0.1524" layer="91"/>
-</segment>
-</net>
-<net name="N$1" class="0">
-<segment>
-<pinref part="JP6" gate="G$1" pin="47/CAPRETURN1"/>
-<wire x1="530.86" y1="144.78" x2="533.4" y2="144.78" width="0.1524" layer="91"/>
-<pinref part="R26" gate="G$1" pin="2"/>
-</segment>
-</net>
-<net name="N$2" class="0">
-<segment>
-<pinref part="JP6" gate="G$1" pin="31/CAPRETURN2"/>
-<pinref part="R27" gate="G$1" pin="2"/>
-<wire x1="530.86" y1="185.42" x2="533.4" y2="185.42" width="0.1524" layer="91"/>
 </segment>
 </net>
@@
 </schematic>
 </drawing>
+<compatibility>
+<note version="6.3" minversion="6.2.2" severity="warning">
+Since Version 6.2.2 text objects can contain more than one line,
+which will not be processed correctly with this version.
+</note>
+</compatibility>
 </eagle>
