File: HARDWARE/The Flying Jalapeno.sch (EAGLE design)
At the start: 97 parts, among them Q2 MMBT2222A, Q3 NDP6020P, Q4 MMBT2222A, Q5 NDP6020P, Q6 BSS138, 200mA/50V, Q7 BSS138, 200mA/50V, U1 ATMEGA2560AU, U2 LM1117, U3 LM1117, U4 LM1117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

Commit message: incremented version number to v10
in sch and brd
Had to nudge traces around when I replaced the fj connector for the
updated package.
Other:
- note added: "v10"
- note removed: "v02"
Changed lines of the file:
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@@
 <text x="200.66" y="269.24" size="3.81" layer="97">MICRO</text>
 <text x="354.33" y="11.43" size="2.54" layer="94">Pete Lewis</text>
-<text x="422.402" y="7.62" size="2.54" layer="94">v02</text>
+<text x="422.402" y="7.62" size="2.54" layer="94">v10</text>
 <text x="284.48" y="96.52" size="1.778" layer="97">ATMEGA2560V</text>
 <text x="457.2" y="246.38" size="3.81" layer="97">2x30 RA connector to testbeds</text>
